File: Eagle files/Tdog v0.9.sch (EAGLE design)
At the start: 115 parts, among them IC1 LM358D, IC2 741G53DCT, IC3 MAX4310EUA, J1 AVR_SPI_PRG_6NS, Q1 27MHz, U1 ATMEGA328P, Y1 16MHz

Commit message: some more connectors
Parts:
- removed OSD_TX: (no value), switch-dil:DS01E
- removed Y1: 16MHz, SparkFun:RESONATORSMD
- added C15: (no value), rcl:C-EUC1206
- added C25: 22pF, SparkFun:CAP0402-CAP
- added C29, C31, C33, C34, C35, C41, C42, C43, C44, C45, C46: 0.1uF, SparkFun:CAP0402-CAP
- added C32: o.1uF, SparkFun:CAP0402-CAP
- added C36, C37: (no value), rcl:CPOL-EUE3.5-10
- added C38, C39, C40, C47: 100pF, SparkFun:CAP0402-CAP
- added IC4: LM358D, linear:LM358D
- added IC5: MAX4310EUA, maxim:MAX4310EUA
- added J$5, J$6: SMA_EDGE, 3DRobotics:SMA_EDGE
- added JP4, JP8: (no value), con-subd:F09H
- added L10, L11, L12, L14, L15, L16, L17, L3, L6, L7, L8, L9: BLM15HD102SN1, pel_dipol_comp:INDUCTOR-0402
- added L13: BKP1005HS121-T, pel_dipol_comp:INDUCTOR-0402
- added LED1: GREEN, SparkFun:LED0603
- added LED2: RED, SparkFun:LED0603
- added OSD_TX1, OSD_TX2: (no value), switch-dil:DS01E
- added Q2: 16MHz, special:XTAL/S
- added R24, R25: 4.7k, SparkFun:RESISTOR0402-RES
- added R38: 0, SparkFun:RESISTOR0402-RES
- added R39: -, SparkFun:RESISTOR0402-RES
- added R40, R41, R42: 75, SparkFun:RESISTOR0402-RES
- added R43: 1k, SparkFun:RESISTOR0402-RES
- added R44, R45: 330, SparkFun:RESISTOR0402-RES
- added SERIAL1, SERIAL2, SERIAL3: (no value), SparkFun:M06SIP
- added SJ3: (no value), jumper:SJ2WW
- added SV1: (no value), con-lstb:MA04-1
- added SV2, SV3, SV4: (no value), con-lstb:MA12-1
- added U$18: DF13-5P-1.25DSA, pixhawk2:DF13-5P-1.25DSA
- added U$19: DF13-4P-1.25DSA, pixhawk2:DF13-4P-1.25DSA
- added U$6, U$8: BOSCMARX5808, boscam:BOSCMARX5808
- added U2: ATMEGA2560-16AU, Atmel_By_element14_Batch_1-00:ATMEGA2560-16AU
- added U4: MAX232, SparkFun:MAX232SOIC16
- added X1: USB-A-H, SparkFun:USB-A-H
- C23: value 0.1uF -> 22pF
- R19: value 10k -> 1k
- R22: value 4.7k -> 10k
- R23: value 15k -> 4.7k
- U1: value ATMEGA328P -> FT232RL-BASICSSOP; device SparkFun:ATMEGA168 -> SparkFun:FT232RL-BASICSSOP
Connections:
- net CH1 renamed CH1_A
- net CH2 renamed CH2_A
- net CH3 renamed CH3_A
- new net 1: C36.+, C37.+, C39.2, C40.2, SJ3.2
- new net ANALOG_5: SV4.11, U2.PF5_(ADC5/TMS)
- new net ANALOG_6: SV4.12, U2.PF6_(ADC6/TDO)
- new net CH1_A_LED: R10.2, U2.PK0_(ADC8/PCINT16)
- new net CH1_B: R23.1
- new net CH1_B_LED: R23.2, U2.PK3_(ADC11/PCINT19)
- new net CH2_A_LED: R11.2, U2.PK1_(ADC9/PCINT17)
- new net CH2_B: R24.1
- new net CH2_B_LED: R24.2, U2.PK4_(ADC12/PCINT20)
- new net CH3_A_LED: R26.2, U2.PK2_(ADC10/PCINT18)
- new net CH3_B: R25.1
- new net CH3_B_LED: R25.2, U2.PK5_(ADC13/PCINT21)
- new net D22: SV2.4, U2.PA0_(AD0)
- new net D23: SV2.5, U2.PA1_(AD1)
- new net D24: SV2.6, U2.PA2_(AD2)
- new net D25: SV2.7, U2.PA3_(AD3)
- new net D26: SV2.8, U2.PA4_(AD4)
- new net D27: SV2.9, U2.PA5_(AD5)
- new net D28: SV2.10, U2.PA6_(AD6)
- new net D29: SV2.11, U2.PA7_(AD7)
- new net D30: SV2.12, U2.PC7_(A15)
- new net D31: SV3.4, U2.PC6_(A14)
- new net D32: SV3.5, U2.PC5_(A13)
- new net D33: SV3.6, U2.PC4_(A12)
- new net D34: SV3.7, U2.PC3_(A11)
- new net D35: SV3.8, U2.PC2_(A10)
- new net D36: SV3.9, U2.PC1_(A9)
- new net D37: SV3.10, U2.PC0_(A8)
- new net D42: SV3.11, U2.PL7
- new net D43: SV3.12, U2.PL6
- new net D44: SV4.4, U2.OC5C)_PL5
- new net D45: SV4.5, U2.(OC5B)_PL4
- new net D46: SV4.6, U2.(OC5A)_PL3
- new net D47: SV4.7, U2.(T5)_PL2
- new net D48: SV4.8, U2.(ICP5)_PL1
- new net D49: SV4.10, SV4.9, U2.(ICP4)_PL0
- new net N$24: OSD_TX1.2, U2.(TXD0)_PE1
- new net N$46: IC4A.+IN
- new net N$48: IC5.IN0, R41.2
- new net N$49: IC5.IN1, R40.2
- new net N$50: IC5.FB, R38.2, R39.1
- new net N$53: L9.2, SERIAL2.2
- new net N$54: J$6.SIGNAL, U$6.P$11
- new net N$56: L10.2, SERIAL2.3
- new net N$57: L8.2, SERIAL1.3
- new net N$58: L11.2, SERIAL3.2
- new net N$61: L12.2, SERIAL3.3
- new net N$62: C41.1, U1.3V3OUT, U1.VCCIO
- new net N$63: U1.USBDP, X1.D-
- new net N$64: U1.USBDM, X1.D+
- new net N$65: LED2.A, R45.1
- new net N$66: LED1.A, R44.1
- new net N$67: LED2.C, U1.TXLED
- new net N$68: LED1.C, U1.RXLED
- new net N$69: L13.1, X1.GND
- new net N$70: L3.1, OSD_TX2.1
- new net N$71: C45.1, U4.V+
- new net N$72: C45.2, U4.V-
- new net N$73: C44.1, U4.C2+
- new net N$74: C44.2, U4.C2-
- new net N$75: C43.1, U4.C1+
- new net N$76: JP4.3, U4.R1IN
- new net N$77: JP4.2, U4.T1OUT
- new net N$78: C43.2, U4.C1-
- new net N$80: L17.2, U4.T1IN
- new net N$81: L14.2, U4.T2IN
- new net N$82: L15.2, U4.R1OUT
- new net N$83: L16.2, U4.R2OUT
- new net N$84: JP8.2, U4.T2OUT
- new net N$85: JP8.3, U4.R2IN
- new net RSSI2: IC4A.-IN, IC4A.OUT, U2.PF2_(ADC2)
- new net RSSI3: IC4B.-IN, IC4B.OUT, U2.PF3_(ADC3)
- new net RX1: L8.1, U$18-2.S, U2.(TXD1/INT3)_PD3
- new net RX2: L10.1, L15.1, U2.(TXD2)_PH1
- new net RX3: L12.1, L16.1, U2.PJ1_(TXD3/PCINT10)
- new net SCL: SV1.2, U$19-2.S, U2.(SCL/INT0)_PD0
- new net SDA: SV1.1, U$19-3.S, U2.(SDA/INT1)_PD1
- new net SHUTDOWN0: IC3.!SHDN, R19.1, U2.(TOSC1)_PG4
- new net SHUTDOWN1: IC5.!SHDN, R43.1, U2.(TOSC2)_PG3
- new net TX1: L7.1, U$18-3.S, U2.(RXD1/INT2)_PD2
- new net TX12: L9.1
- new net TX2: L17.1, U2.(RXD2)_PH0
- new net TX3: L11.1, L14.1, U2.PJ0_(RXD3/PCINT9)
- new net VCC: U$18-1.S
- new net XTAL1: C23.2, Q2.1, U2.XTAL1
- new net XTAL2: C25.1, Q2.2, U2.XTAL2
- net 3.3V: now also SJ3.3, SV2.3, SV3.3, SV4.3, U$19-1.S
- net 5V: now also C29.2, C31.2, C32.2, C33.2, C34.2, C35.2, C38.2, C42.1, C46.1, C47.2, IC4P.V+, IC5.V+, L13.2, R44.2, R45.2, SERIAL1.4, SERIAL2.4, SERIAL3.4, SJ3.1, SV1.3, SV2.2, SV3.2, SV4.2, U1.VCC, U2.AREF, U2.AVCC, U2.VCC, U2.VCC_2, U2.VCC_3, U2.VCC_4, U4.VCC; no longer R19.2, R23.1, U1.AVCC, U1.VCC@1, U1.VCC@2
- net 5V_SERVO: now also C15.2; no longer C23.2
- net CH1_LED: no longer R10.2, U1.PB0(ICP)
- net CH2_LED: no longer R11.2, U1.PB1(OC1A)
- net CH3_LED: no longer R26.2, U1.PB2(SS/OC1B)
- net CTS: now also U1.CTS
- net DTR: now also U1.DTR
- net GND: now also C23.1, C25.2, C29.1, C31.1, C32.1, C33.1, C34.1, C35.1, C36.-, C37.-, C38.1, C39.1, C40.1, C41.2, C42.2, C46.2, C47.1, IC4P.V-, IC5.V-, J$5.GND@0, J$5.GND@1, J$5.GND@2, J$5.GND@3, J$6.GND@0, J$6.GND@1, J$6.GND@2, J$6.GND@3, JP4.5, JP8.5, R19.2, R39.2, R40.1, R41.1, R42.2, R43.2, SERIAL1.5, SERIAL1.6, SERIAL2.5, SERIAL2.6, SERIAL3.5, SERIAL3.6, SV1.4, SV2.1, SV3.1, SV4.1, U$18-5.S, U$19-4.S, U$6.P$10, U$6.P$12, U$8.P$10, U$8.P$12, U1.GND1, U1.GND2, U1.GND3, U1.TEST, U2.GND, U2.GND_2, U2.GND_3, U2.GND_4, U2.GND_5, U4.GND, X1.VBUS; no longer U1.GND@1, U1.GND@2, Y1.2
- net MISO: now also U2.(MISO/PCINT3)_PB3; no longer U1.PB4(MISO)
- net MOSI: now also U2.(MOSI/PCINT2)_PB2; no longer U1.PB3(MOSI/OC2)
- net N$2: now also BLUETOOTH_HC-05.2, L3.2; no longer R23.2, U1.AREF
- net N$3: now also BLUETOOTH_HC-05.3, L6.2; no longer U1.PB6(XTAL1/TOSC1), Y1.1
- net N$36: now also IC4B.+IN; no longer IC3.!SHDN, R19.1
- net N$4: now also L7.2, SERIAL1.2; no longer U1.PB7(XTAL2/TOSC2), Y1.3
- net N$55: now also J$5.SIGNAL, U$8.P$11; no longer OSD_TX.2, U1.PD1(TXD)
- net PAN_SERVO: now also U2.(OC1A/PCINT5)_PB5; no longer U1.PD5(T1)
- net RESET: now also U2.~RESET; no longer U1.PC6(/RESET)
- net RSSI0: now also U2.PF0_(ADC0); no longer U1.PC0(ADC0)
- net RSSI1: now also U2.PF1_(ADC1); no longer U1.PC1(ADC1)
- net RTS: now also U1.RTS
- net RX: now also L6.1, OSD_TX1.1, U1.TXD; no longer BLUETOOTH_HC-05.3, OSD_TX.1
- net SCK: now also U2.(SCK/PCINT1)_PB1; no longer U1.PB5(SCK)
- net SERVO_GND: now also C15.1; no longer C23.1
- net SSOSD-IN: now also U2.(OC4A)_PH3; no longer U1.PD6(AIN0)
- net SWITCH0: now also U2.PG2_(ALE); no longer U1.PD3(INT1)
- net TILT_SERVO: now also U2.(OC1B/PCINT6)_PB6; no longer U1.PD7(AIN1)
- net TX: now also OSD_TX2.2, U1.RXD, U2.(RXD0/PCINT8)_PE0; no longer BLUETOOTH_HC-05.2, U1.PD0(RXD)
- net VIDEO_MUX: now also IC5.A0, U2.(OC0B)_PG5; no longer U1.PD4(XCK/T0)
- net VIDEO_SWITCHED: now also IC5.OUT, R38.1, R42.1
- net VIN_SENS: now also U2.PF4_(ADC4/TCK); no longer U1.PC2(ADC2)
- net VSYNC: now also U2.(OC3B/INT4)_PE4; no longer U1.PD2(INT0)
Other:
- moved on the sheet: BLUETOOTH_HC-05, C1, C10, C11, C12, C13, C14, C16, C17, C18, C19, C2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
